File: Hardware/SparkFun_USDA_Watershed_Monitor.brd (EAGLE design)
At the start: 63.5 x 63.5 mm, 194 parts, among them J10 QWIIC_RIGHT_ANGLE, J3 QWIIC_RIGHT_ANGLE, J4 U.FL, J5 RJ45, J7 RJ45, J9 RJ45, Q1 20V/4.2A/52mΩ/1.4W, Q2 20V/0.2A/8MHz/1.2Ω/1Vth, Q3 20V/0.2A/8MHz/1.2Ω/1Vth, Q4 20V/0.2A/8MHz/1.2Ω/1Vth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

Commit message: Move load cell connector to bottom edge
Will help a lot with panelization
Moved left GPIO RJ45 connector to bottom middle, and redid connections for easier routing
Parts:
- removed U$49, U$51: (no value), output:#_3V3#0
- removed U$50, U$53: (no value), output:#_GND#0
- added U$56: (no value), output:#SCL_#0
- added U$81: (no value), output:#_SCL#1
- added U$84: (no value), output:#_SDA#2
- added U$85: (no value), output:#_3V3#0
- U$47: device output:#_IO26#0 -> output:#3V3_#0
- U$48: device output:#_IO27#0 -> output:#SDA_#0
- U$6: device output:#_IO26#0 -> output:#GND_#0
- U$7: device output:#_IO27#0 -> output:#_GND#0
- moved U$52 69.5 mm to (81.9, 16.0)
- moved U$62 69.5 mm to (81.9, 14.5)
- moved U$64 69.5 mm to (81.9, 17.5)
- moved U$54 69.5 mm to (85.7, 14.5)
- moved U$61 69.5 mm to (85.7, 16.0)
- moved U$63 69.5 mm to (85.7, 17.5)
- moved U$32 55.5 mm to (87.0, 27.7)
- moved U$33 55.5 mm to (83.2, 27.7)
- moved U$34 55.5 mm to (87.0, 26.2)
- moved U$35 55.5 mm to (83.2, 26.2)
- moved U$36 55.5 mm to (87.0, 24.6)
- moved U$37 55.5 mm to (83.2, 24.6)
- moved U$38 55.5 mm to (87.0, 23.1)
- moved U$39 55.5 mm to (83.2, 23.1)
- moved U$45 55.5 mm to (85.1, 29.2)
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Connections:
- net ESP_I35: now also J7.1; no longer J7.4
- net ESP_I36: now also J7.5; no longer J7.1
- net ESP_I39: now also J7.6; no longer J7.2
- net ESP_IO25: now also J7.2; no longer J7.6
- net ESP_IO26: no longer J8.1
- net ESP_IO27: no longer J8.2
- net ESP_IO33: now also J7.4; no longer J7.5
- net SCL: now also J8.1
- net SDA: now also J8.2
Routing:
- net ESP_IO26: track 48.2 -> 1.67 mm
- net ESP_IO27: track 47.6 -> 1.67 mm
- net ESP_I39: track 52.8 -> 66.5 mm
- net ESP_I36: track 56.2 -> 65.8 mm
- net SCL: track 132.3 -> 141.7 mm
- net SDA: track 124.2 -> 133.0 mm, vias 9 -> 10
- net NAU_INT: track 27.8 -> 35.3 mm
- net ESP_I34: track 54.7 -> 58.8 mm
- net 3.3V: track 265.3 -> 267.7 mm
- net GND: track 21.3 -> 22.8 mm, vias 270 -> 259
- net NAU_B+: track 16.1 -> 14.8 mm
- net ESP_IO33: track 55.7 -> 56.8 mm
- net ESP_I35: track 51.9 -> 53.0 mm
- net ESP_IO25: track 53.1 -> 52.2 mm
- net NAU_A+: track 4.91 -> 4.14 mm
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